File: keypad_pcb_surface_mount/merch-hat.brd (EAGLE design)
At the start: 65 x 56 mm, 29 parts, among them U2 ATMEGA328P_TQFP, Y2 16MHZ

Commit message: Minor fixes
Parts:
- moved C1 1.91 mm to (17.8, 27.6)
Routing:
- net SCK: track 13.0 -> 11.8 mm
Other:
- board text added: "Merch v0.2"
Changed lines of the file:
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@@
 <text x="11.811" y="30.48" size="1.27" layer="21">INT</text>
 <text x="11.811" y="28.067" size="1.27" layer="21">XSHD</text>
+<text x="46.863" y="6.35" size="1.778" layer="21">Merch v0.2</text>
 </plain>
 <attributes>
@@
 </element>
 <element name="PORT" library="pinhead" package="1X03" value="Sensor Port" x="61.468" y="44.704" smashed="yes" rot="R270">
-<attribute name="NAME" x="58.3438" y="47.4472" size="1.27" layer="25" ratio="10" rot="R270"/>
+<attribute name="NAME" x="64.2112" y="40.4622" size="1.27" layer="25" ratio="10" rot="R180"/>
 <attribute name="VALUE" x="58.293" y="48.514" size="1.27" layer="27" rot="R270"/>
 </element>
@@
 <attribute name="VALUE" x="25.908" y="32.893" size="1.27" layer="27" rot="R180"/>
 </element>
-<element name="C1" library="SparkFun-Capacitors" package="0603-CAP" value="0.1uF" x="15.875" y="27.559" rot="R90"/>
+<element name="C1" library="SparkFun-Capacitors" package="0603-CAP" value="0.1uF" x="17.78" y="27.559" rot="R90"/>
 <element name="R12" library="resistor" package="R0805" value="3.3k" x="30.226" y="37.465" smashed="yes" rot="R180">
 <attribute name="NAME" x="31.623" y="36.195" size="1.27" layer="25" rot="R180"/>
@@
 <wire x1="8.382" y1="48.26" x2="6.731" y2="48.26" width="0.4064" layer="1"/>
 <wire x1="6.731" y1="48.26" x2="6.731" y2="26.416" width="0.4064" layer="1"/>
-<wire x1="15.875" y1="26.416" x2="6.731" y2="26.416" width="0.4064" layer="1"/>
+<wire x1="17.78" y1="26.416" x2="18.923" y2="26.416" width="0.4064" layer="1"/>
 <via x="18.923" y="26.416" extent="1-16" drill="0.6"/>
-<wire x1="15.875" y1="26.416" x2="18.923" y2="26.416" width="0.4064" layer="1"/>
+<wire x1="17.78" y1="26.416" x2="6.731" y2="26.416" width="0.4064" layer="1"/>
 <wire x1="18.923" y1="26.416" x2="21.209" y2="26.416" width="0.4064" layer="16"/>
 <wire x1="21.209" y1="26.416" x2="21.209" y2="16.707" width="0.4064" layer="16"/>
 <wire x1="21.209" y1="26.416" x2="24.511" y2="26.416" width="0.4064" layer="16"/>
 <via x="24.511" y="26.416" extent="1-16" drill="0.6"/>
-<wire x1="28.575" y1="30.48" x2="31.75" y2="33.655" width="0.4064" layer="1"/>
-<wire x1="28.575" y1="30.48" x2="24.511" y2="26.416" width="0.4064" layer="1"/>
+<wire x1="28.448" y1="30.353" x2="31.75" y2="33.655" width="0.4064" layer="1"/>
+<wire x1="28.448" y1="30.353" x2="24.511" y2="26.416" width="0.4064" layer="1"/>
 <wire x1="31.75" y1="33.655" x2="32.766" y2="33.655" width="0.4064" layer="1"/>
 <via x="32.766" y="33.655" extent="1-16" drill="0.6"/>
@@
 <contactref element="R11" pad="1"/>
 <contactref element="C1" pad="1"/>
-<wire x1="15.875" y1="26.709" x2="15.875" y2="26.416" width="0.4064" layer="1"/>
 <contactref element="R12" pad="1"/>
 <contactref element="R13" pad="1"/>
 <wire x1="35.748" y1="42.799" x2="35.748" y2="41.463" width="0.4064" layer="1"/>
 <wire x1="33.782" y1="39.497" x2="35.748" y2="41.463" width="0.4064" layer="1"/>
-<via x="33.782" y="39.497" extent="1-16" drill="0.6" shape="square"/>
+<via x="33.782" y="39.497" extent="1-16" drill="0.6"/>
 <wire x1="33.782" y1="39.497" x2="33.782" y2="34.671" width="0.4064" layer="16"/>
 <wire x1="33.782" y1="34.671" x2="32.766" y2="33.655" width="0.4064" layer="16"/>
@@
 <wire x1="31.75" y1="37.465" x2="33.782" y2="39.497" width="0.4064" layer="1"/>
 <wire x1="26.223" y1="30.353" x2="28.448" y2="30.353" width="0.4064" layer="1"/>
-<wire x1="28.448" y1="30.353" x2="28.575" y2="30.48" width="0.4064" layer="1"/>
+<wire x1="17.78" y1="26.709" x2="17.78" y2="26.416" width="0.4064" layer="1"/>
 <wire x1="8.382" y1="48.26" x2="9.652" y2="48.26" width="0" layer="19" extent="1-16"/>
 </signal>
@@
 <contactref element="GPIO1" pad="34"/>
 <contactref element="C1" pad="2"/>
-<via x="13.716" y="28.702" extent="1-16" drill="0.6" shape="square"/>
-<via x="17.78" y="28.321" extent="1-16" drill="0.6" shape="square"/>
+<via x="15.367" y="28.321" extent="1-16" drill="0.6"/>
+<via x="20.193" y="28.067" extent="1-16" drill="0.6"/>
 </signal>
 <signal name="GPIO20">
@@
 <contactref element="LCD" pad="10"/>
 <wire x1="9.271" y1="21.463" x2="11.811" y2="21.463" width="0.4064" layer="1"/>
-<wire x1="11.811" y1="21.463" x2="16.637" y2="21.463" width="0.4064" layer="16"/>
-<wire x1="16.637" y1="21.463" x2="18.923" y2="23.749" width="0.4064" layer="16"/>
-<via x="18.923" y="23.749" extent="1-16" drill="0.6"/>
-<wire x1="18.923" y1="23.749" x2="19.1456" y2="23.749" width="0.4064" layer="1"/>
-<wire x1="19.1456" y1="23.749" x2="20.695" y2="22.1996" width="0.4064" layer="1"/>
+<wire x1="20.695" y1="22.1996" x2="19.304" y2="22.1996" width="0.4064" layer="1"/>
+<wire x1="19.304" y1="22.1996" x2="19.304" y2="22.225" width="0.4064" layer="1"/>
+<via x="19.304" y="22.225" extent="1-16" drill="0.6"/>
+<wire x1="19.304" y1="22.225" x2="18.542" y2="21.463" width="0.4064" layer="16"/>
+<wire x1="18.542" y1="21.463" x2="11.811" y2="21.463" width="0.4064" layer="16"/>
 </signal>
 <signal name="IO7">
