File: keypad_pcb_surface_mount/merch-hat.brd (EAGLE design)
At the start: 65 x 56 mm, 34 parts, among them U1 CAT24C32, U2 ATMEGA328P_TQFP, Y2 16MHZ

Commit message: add power connctor, new range sensor pinout, pullup
Parts:
- removed VL53L0X: VL53L0X, pinhead:1X06
- added +5V: (no value), con-jack:SPC4078
- added CUP: (no value), pinhead:1X07
- added R17: 1.5K, rcl:R0603
Connections:
- new net N$3: PORT_OUT.2, R17.1
- net +5V: now also +5V.3, CUP.1; no longer VL53L0X.1
- net GND: now also +5V.1, CUP.3; no longer VL53L0X.2
- net GPIO2: now also CUP.7; no longer VL53L0X.4
- net GPIO20: now also R17.2
- net GPIO3: now also CUP.6; no longer VL53L0X.3
- net GPIO4: now also CUP.4; no longer VL53L0X.5
Routing:
- net GPIO2: track 23.2 -> 8.33 mm
- net GPIO4: track 26.5 -> 18.3 mm
- net GPIO3: track 18.8 -> 12.1 mm
- net GPIO20: track 8.31 -> 13.4 mm
- net N$3: track 0.00 -> 4.95 mm
- net GPIO6: track 49.8 -> 49.0 mm
Other:
- board text added: "GPIO"
- board text added: "Merch v1"
- board text removed: "10"
- board text removed: "BOTTOM"
- board text removed: "INT"
- board text removed: "Merch v0.2"
- board text removed: "TOP"
- board text removed: "XSHD"
